Commit message: Fix rotated point cloud

File: si_bot/urdf/si_bot.xacro (robot description, xacro)
@@ -432,4 +432,11 @@
     </visual>
   </link>
+  <!-- Fix for rotated point cloud -->
+  <joint name="camera_link_joint" type="fixed">
+    <origin xyz="0 0 0" rpy="-1.5707 0 -1.5707" />
+    <child link="camera_link" />
+    <parent link="camera" />
+  </joint>
+  <link name="camera_link"></link>
   <!-- ======= Laser Rangefinder ======= -->
   <!--

Commit message: Fix laer scan

File: si_bot/urdf/si_bot.xacro (robot description, xacro)
@@ -465,5 +465,5 @@
       <geometry>
         <mesh filename="package://si_bot/meshes/hokuyo.dae" />
-        <box size="0.1 0.1 0.1" />
+        <!-- <box size="0.1 0.1 0.1" /> -->
       </geometry>
     </visual>
